File: design/board.kicad_pcb (KiCad board)
At the start: 2 copper layers, 96.5 x 81.3 mm, 14 parts, among them J1 Mic, J2 DEBUG_CONN, J3 PWR_CONN, J4 0.97" OLED, J5 WS2812b, SW1 SW_Push, U1 NodeMCU1.0(ESP-12E), U2 BME280

Commit message: added some Text on Silkscreen and some holes
Parts:
- moved D1 3.05 mm to (90.9, 22.9)
Routing:
- net Net-(D1-Pad2): track 19.6 -> 17.2 mm
- net VCC: track 270.6 -> 269.3 mm
Other:
- outline, holes or cut-outs redrawn
- board text added: "+"
- board text added: "-"
- board text added: "3.3V 5V GND SDA SCL WS2812B MIC"
- board text added: "3.3V GND SCL SDA CSB SDO"
- board text added: "5V DATA OUT GND"
- board text added: "GND 5V SDA SCL"
- board text added: "OFF"
- board text added: "ON"
- board text added: "VCC GND MIC"
Changed lines of the file:
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@@
 (kicad_pcb (version 4) (host pcbnew 4.0.6)
   (general
-    (links 0)
-    (no_connects 4)
+    (links 41)
+    (no_connects 0)
     (area 20.244999 15.164999 116.915001 96.595001)
     (thickness 1.6)
-    (drawings 7)
-    (tracks 124)
+    (drawings 22)
+    (tracks 126)
     (zones 0)
     (modules 14)
@@
     (descr "Through hole straight pin header, 1x03, 2.54mm pitch, single row")
     (tags "Through hole pin header THT 1x03 2.54mm single row")
-    (fp_text reference JP1 (at 0 -2.33 90) (layer F.SilkS)
+    (fp_text reference JP1 (at 2.032 2.54 180) (layer F.SilkS)
       (effects (font (size 1 1) (thickness 0.15)))
     )
@@
     (descr "Through hole straight pin header, 1x03, 2.54mm pitch, single row")
     (tags "Through hole pin header THT 1x03 2.54mm single row")
-    (fp_text reference JP2 (at 0 -2.33 90) (layer F.SilkS)
-      (effects (font (size 1 1) (thickness 0.15)))
-    )
-    (fp_text value BEEPER_JUMP (at -3.556 3.048 180) (layer F.SilkS)
+    (fp_text reference JP2 (at -2.54 2.54 180) (layer F.SilkS)
+      (effects (font (size 1 1) (thickness 0.15)))
+    )
+    (fp_text value BEEPER_JUMP (at -4.572 3.048 180) (layer F.SilkS)
       (effects (font (size 1 1) (thickness 0.15)))
     )
@@
       (effects (font (size 1 1) (thickness 0.15)))
     )
-    (fp_text value SW_Push (at 0 4.87) (layer F.Fab)
+    (fp_text value SW_Push (at 0 4.87) (layer F.SilkS)
       (effects (font (size 1 1) (thickness 0.15)))
     )
@@
   )
   (module Diodes_THT:D_DO-201AD_P15.24mm_Horizontal (layer F.Cu)
-    (at 93.98 22.86)
+    (at 90.932 22.86)
     (descr "D, DO-201AD series, Axial, Horizontal, pin pitch=15.24mm, , length*diameter=9.5*5.2mm^2, , http://www.diodes.com/_files/packages/DO-201AD.pdf")
     (tags "D DO-201AD series Axial Horizontal pin pitch 15.24mm  length 9.5mm diameter 5.2mm")
@@
     )
   )
-  (gr_text "Mainframe - Ferienpass 2017" (at 112.776 74.168 90) (layer F.SilkS)
+  (gr_text "VCC\nGND\nMIC" (at 90.678 64.008) (layer F.SilkS)
+    (effects (font (size 1.5 1.5) (thickness 0.3)))
+  )
+  (gr_text OFF (at 53.34 86.36) (layer F.SilkS)
+    (effects (font (size 1.5 1.5) (thickness 0.3)))
+  )
+  (gr_text OFF (at 53.34 80.518) (layer F.SilkS)
+    (effects (font (size 1.5 1.5) (thickness 0.3)))
+  )
+  (gr_text ON (at 66.04 86.614) (layer F.SilkS)
+    (effects (font (size 1.5 1.5) (thickness 0.3)))
+  )
+  (gr_text ON (at 65.786 80.264) (layer F.SilkS)
+    (effects (font (size 1.5 1.5) (thickness 0.3)))
+  )
+  (gr_text "GND\n5V\nSDA\nSCL" (at 39.37 60.198) (layer F.SilkS)
+    (effects (font (size 1.5 1.5) (thickness 0.3)))
+  )
+  (gr_text "3.3V\nGND\nSCL\nSDA\nCSB\nSDO" (at 24.384 62.738) (layer F.SilkS)
+    (effects (font (size 1.5 1.5) (thickness 0.3)))
+  )
+  (gr_text "5V\nDATA OUT\nGND\n" (at 29.972 36.068) (layer F.SilkS)
+    (effects (font (size 1.5 1.5) (thickness 0.3)) (justify left))
+  )
+  (gr_text "3.3V\n5V\nGND\nSDA\nSCL\nWS2812B\nMIC" (at 44.704 38.608) (layer F.SilkS)
+    (effects (font (size 1.5 1.5) (thickness 0.3)) (justify left))
+  )
+  (gr_text - (at 96.52 33.528) (layer F.SilkS)
+    (effects (font (size 1.5 1.5) (thickness 0.3)))
+  )
+  (gr_text + (at 95.504 30.988) (layer F.SilkS)
+    (effects (font (size 1.5 1.5) (thickness 0.3)) (justify left))
+  )
+  (gr_circle (center 25.4 20.32) (end 26.9 20.32) (layer Edge.Cuts) (width 0.15))
+  (gr_circle (center 111.76 20.32) (end 113.29 20.32) (layer Edge.Cuts) (width 0.15))
+  (gr_circle (center 111.76 91.44) (end 113.26 91.44) (layer Edge.Cuts) (width 0.15))
+  (gr_circle (center 25.4 91.44) (end 26.9 91.44) (layer Edge.Cuts) (width 0.15))
+  (gr_text "Mainframe - Ferienpass 2017" (at 112.776 58.928 90) (layer F.SilkS)
     (effects (font (size 1.5 1.5) (thickness 0.3)))
   )
@@
   (segment (start 28.448 55.238) (end 28.448 56.388) (width 0.3) (layer F.Cu) (net 3))
   (segment (start 43.18 30.988) (end 56.896 30.988) (width 0.3) (layer F.Cu) (net 3))
+  (segment (start 90.932 22.86) (end 90.932 24.76) (width 0.3) (layer F.Cu) (net 4))
+  (segment (start 90.932 24.76) (end 87.752 27.94) (width 0.3) (layer F.Cu) (net 4))
+  (segment (start 87.752 27.94) (end 87.752 30.988) (width 0.3) (layer F.Cu) (net 4))
   (segment (start 88.9 32.512) (end 94.488 38.1) (width 0.3) (layer B.Cu) (net 4))
   (via (at 94.488 40.64) (size 0.6) (drill 0.4) (layers F.Cu B.Cu) (net 4))
@@
   (segment (start 108.712 34.036) (end 107.188 35.56) (width 0.3) (layer F.Cu) (net 4))
   (segment (start 99.568 35.56) (end 94.488 40.64) (width 0.3) (layer F.Cu) (net 4))
-  (segment (start 93.98 22.86) (end 93.98 24.76) (width 0.3) (layer F.Cu) (net 4))
-  (segment (start 93.98 24.76) (end 87.752 30.988) (width 0.3) (layer F.Cu) (net 4))
   (segment (start 87.752 30.988) (end 85.91363 30.988) (width 0.3) (layer F.Cu) (net 4))
   (segment (start 85.91363 30.988) (end 84.836 30.988) (width 0.3) (layer F.Cu) (net 4))
@@
   (segment (start 51.308 56.388) (end 52.458 56.388) (width 0.3) (layer F.Cu) (net 14))
   (segment (start 52.458 56.388) (end 56.896 56.388) (width 0.3) (layer F.Cu) (net 14))
-  (segment (start 109.22 22.86) (end 101.092 30.988) (width 0.3) (layer F.Cu) (net 30))
-  (segment (start 101.092 30.988) (end 93.98 30.988) (width 0.3) (layer F.Cu) (net 30))
+  (segment (start 106.172 22.86) (end 100.958 22.86) (width 0.3) (layer F.Cu) (net 30))
+  (segment (start 100.958 22.86) (end 93.98 29.838) (width 0.3) (layer F.Cu) (net 30))
+  (segment (start 93.98 29.838) (end 93.98 30.988) (width 0.3) (layer F.Cu) (net 30))
   (segment (start 94.996 30.988) (end 93.98 30.988) (width 0.3) (layer B.Cu) (net 30))
   (zone (net 2) (net_name GND) (layer F.Cu) (hatch edge 0.508)
     (connect_pads (clearance 0.508))
     (min_thickness 0.254)
-    (fill (arc_segments 16) (thermal_gap 0.508) (thermal_bridge_width 0.508))
+    (fill yes (arc_segments 16) (thermal_gap 0.508) (thermal_bridge_width 0.508))
     (polygon
       (pts
@@
     (connect_pads (clearance 0.508))
     (min_thickness 0.254)
-    (fill (arc_segments 16) (thermal_gap 0.508) (thermal_bridge_width 0.508))
+    (fill yes (arc_segments 16) (thermal_gap 0.508) (thermal_bridge_width 0.508))
     (polygon
       (pts
